File: RNS.brd (EAGLE design)
At the start: 59.4 x 73.6 mm, 10 parts

Commit message: Add files via upload
Routing:
- net 5V: track 196.8 -> 198.6 mm
Other:
- board size 59.4 x 73.6 mm -> 60.6 x 73.6 mm
Changed lines of the file:
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@@
 <board>
 <plain>
-<wire x1="-2.54" y1="35.56" x2="56.82" y2="35.56" width="0" layer="20"/>
+<wire x1="-3.81" y1="35.56" x2="56.82" y2="35.56" width="0.4064" layer="20"/>
 <wire x1="56.82" y1="35.56" x2="56.82" y2="109.21" width="0.4064" layer="20"/>
-<wire x1="56.82" y1="109.21" x2="-2.54" y2="109.21" width="0.4064" layer="20"/>
-<wire x1="-2.54" y1="109.21" x2="-2.54" y2="35.56" width="0.4064" layer="20"/>
+<wire x1="56.82" y1="109.21" x2="-3.81" y2="109.21" width="0.4064" layer="20"/>
+<wire x1="-3.81" y1="109.21" x2="-3.81" y2="35.56" width="0.4064" layer="20"/>
 </plain>
 <attributes>
@@
 <contactref element="U$2" pad="GND_1"/>
 <contactref element="U$2" pad="GND_2"/>
-<polygon width="1.016" layer="16">
-<vertex x="-3.81" y="110.49"/>
-<vertex x="57.15" y="110.49"/>
+<polygon width="1.016" layer="16" isolate="0.6096">
+<vertex x="-3.81" y="109.22"/>
+<vertex x="57.15" y="109.22"/>
 <vertex x="57.15" y="35.56"/>
 <vertex x="-3.81" y="35.56"/>
@@
 <wire x1="33.02" y1="97.79" x2="33.02" y2="106.68" width="1.016" layer="16"/>
 <wire x1="33.02" y1="106.68" x2="3.81" y2="106.68" width="1.016" layer="16"/>
-<wire x1="3.81" y1="106.68" x2="0.254" y2="103.124" width="1.016" layer="16"/>
-<wire x1="0.254" y1="103.124" x2="0.254" y2="81.28" width="1.016" layer="16"/>
-<wire x1="0.254" y1="81.28" x2="3.81" y2="81.28" width="1.016" layer="16"/>
+<wire x1="3.81" y1="106.68" x2="-1.016" y2="101.854" width="1.016" layer="16"/>
+<wire x1="-1.016" y1="101.854" x2="-1.016" y2="81.28" width="1.016" layer="16"/>
+<wire x1="-1.016" y1="81.28" x2="3.81" y2="81.28" width="1.016" layer="16"/>
 <wire x1="50.8" y1="80.01" x2="50.8" y2="95.25" width="1.016" layer="16"/>
 <wire x1="50.8" y1="95.25" x2="29.21" y2="95.25" width="1.016" layer="16"/>

Commit message: Add files via upload
Parts:
- added +PWR-: (no value), MIA_LIBRARY-2-2-2:1X02
- TTL: device MIA_LIBRARY-2-2-2:1X04/90 -> MIA_LIBRARY-2-2-2:1X04
- moved U$1 10.2 mm to (3.81, 74.9)
- moved TTL 2.54 mm to (52.1, 76.2)
- moved DC-JACK 1.80 mm to (8.89, 101.6)
- moved CYTRON 1.27 mm to (52.1, 63.5)
Connections:
- net 9V renamed 12V
- net 5V: now also +PWR-.1, TTL.2; no longer TTL.1
- net GND: now also +PWR-.2, TTL.1; no longer TTL.2
Routing:
- net 5V: track 198.6 -> 213.3 mm
- net PB_10: track 15.9 -> 12.3 mm
- net PA_9: track 26.5 -> 23.4 mm
- net PA_8: track 26.5 -> 23.4 mm
- net PA_3: track 13.8 -> 11.7 mm
- net 12V: track 20.8 -> 22.6 mm
- net PB_11: track 11.0 -> 12.3 mm
- net PA_2: track 15.2 -> 14.0 mm
Other:
- board size 60.6 x 73.6 mm -> 60.6 x 72.4 mm
