File: RNS.sch (EAGLE design)
At the start: 10 parts

Commit message: Add files via upload
Parts:
- added +PWR-: (no value), MIA_LIBRARY-2-2-2:PINHD-1X2
- TTL: device MIA_LIBRARY-2-2-2:PINHD-1X4/90 -> MIA_LIBRARY-2-2-2:PINHD-1X4
Connections:
- net 9V renamed 12V
- net 5V: now also +PWR-.1, TTL.2; no longer TTL.1
- net GND: now also +PWR-.2, TTL.1; no longer TTL.2
Other:
- moved on the sheet: PWR_LED, U$3
